File: PCB/pico_rx/Lowpass.kicad_sch (KiCad schematic)
At the start: 33 parts, among them J5 Antenna

Commit message: Get CW working
Parts:
- removed C?: 100n, Capacitor_SMD:C_0805_2012Metric, symbol Device:C
- removed J5: Antenna, Connector_Coaxial:SMA_Amphenol_132289_EdgeMount, symbol Connector:Conn_Coaxial
- removed R11, R12: 10K, Resistor_SMD:R_0805_2012Metric, symbol Device:R
Connections:
- net RF_PREAMP: now reaches U?.5 (Y)
