File: PCB/pico_rx/_autosave-qsd.kicad_sch (KiCad schematic)
At the start: 18 parts

Commit message: Get CW working
Other:
- note added: "R, C values determine LPF cutoff 1/(2 * pi * 27e-9 * 100) ~= 59MHz"
- note removed: "R, C values determine LPF cutoff 1/(2 * pi * 27e-9 * 100) ~= 59MHz 1/(2 * pi * 27e-12 * 100000) ~= 59MHz"
Changed lines of the file:
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@@
     (effects (font (size 2.5 2.5)) (justify left bottom))
   )
-  (text "R, C values determine LPF cutoff\n1/(2 * pi * 27e-9 * 100) ~= 59MHz\n1/(2 * pi * 27e-12 * 100000) ~= 59MHz"
-    (at 64.77 35.56 0)
+  (text "R, C values determine LPF cutoff\n1/(2 * pi * 27e-9 * 100) ~= 59MHz"
+    (at 64.77 30.48 0)
     (effects (font (size 2.5 2.5)) (justify left bottom))
   )
