File: PCB/pico_rx/pico_rx.kicad_pcb (KiCad board)
At the start: 2 copper layers, 54.6 x 89.5 mm, 67 parts, among them J1 Speaker, J2 Headphone, J4 I2C Display, J5 Antenna, J6 Battery, SW1 RotaryEncoder_Switch, SW2 SW_Push, SW3 SW_Push, SW4 SW_SPDT, U1 74CBT3251, U2 74CBT3251, U3 LT6231, U4 FST3253, U5 Pico

Commit message: Get CW working
Parts:
- added C10: 100n, Capacitor_SMD:C_0805_2012Metric, F.Cu at (110.5, 122.6)
- added C4: 100p, Capacitor_SMD:C_0805_2012Metric, F.Cu at (120.0, 109.2)
- added C5: 10p, Capacitor_SMD:C_0805_2012Metric, F.Cu at (112.4, 111.8)
- added R1: 50, Resistor_SMD:R_0805_2012Metric, F.Cu at (116.2, 111.8)
- added R11: 500, Resistor_SMD:R_0805_2012Metric, F.Cu at (112.4, 114.3)
- added R12: 0, Resistor_SMD:R_0805_2012Metric, F.Cu at (116.2, 114.3)
- added R13: 1k, Resistor_SMD:R_0805_2012Metric, F.Cu at (104.1, 152.4)
- added R14: 1k, Resistor_SMD:R_0805_2012Metric, F.Cu at (108.0, 152.4)
- added U6: LTC6226xS8, Package_SO:SO-8_3.9x4.9mm_P1.27mm, F.Cu at (112.4, 118.6)
- C26, C27, C28, C29: value 10n -> 27n
- C30, C31: value 47p -> 27p
- R7, R8: value 82K -> 100k
- U3: value LT6231 -> LTC6227
- moved R2 4.97 mm to (120.0, 114.3)
- moved R10 4.89 mm to (120.0, 111.8)
- moved C1 1.59 mm to (116.2, 109.2)
Connections:
- C1 pad 1: Net-(J5-In) -> Net-(C1-Pad1)
- C1 pad 2: Net-(U1-Y) -> Net-(J5-In)
- R10 pad 1: Net-(U1-Y) -> Net-(U6-+)
- R2 pad 2: Net-(U1-Y) -> Net-(U6-+)
- SW1 pad S1: unconnected-(SW1-PadS1) -> /PI Pico/PUSH
- U1 pad 5: Net-(U1-Y) -> RF_PREAMP
- U5 pad 19: /PI Pico/EEPROM_SDA -> unconnected-(U5-GPIO14-Pad19)
- U5 pad 20: /PI Pico/EEPROM_SCL -> unconnected-(U5-GPIO15-Pad20)
- U5 pad 31: RX_Q -> Net-(U5-GPIO26_ADC0)
- U5 pad 32: RX_I -> Net-(U5-GPIO27_ADC1)
- U5 pad 7: unconnected-(U5-GPIO5-Pad7) -> /PI Pico/PUSH
Routing:
- net /PI Pico/PUSH: track 0.00 -> 71.7 mm, vias 0 -> 2
- net Net-(U5-GPIO27_ADC1): track 0.00 -> 47.7 mm
- net RX_I: track 59.1 -> 12.2 mm
- net RF_PREAMP: track 0.00 -> 37.3 mm
- net Net-(U5-GPIO26_ADC0): track 0.00 -> 35.5 mm
- net RX_Q: track 54.8 -> 20.4 mm
- net GND: track 119.4 -> 149.4 mm, vias 248 -> 240
- net Net-(U1-Y): track 25.2 -> 0.00 mm
- net Net-(U6--): track 0.00 -> 22.2 mm
- net Net-(U6-+): track 0.00 -> 15.5 mm
- net +5V: track 203.5 -> 217.3 mm
- net Net-(C1-Pad1): track 0.00 -> 5.10 mm
- net BAND_0: track 117.6 -> 119.5 mm
- net BAND_1: track 119.6 -> 121.2 mm
- net +3V3: track 91.7 -> 92.7 mm
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Other:
- board text added: "!!D1 Must be removed from Pi Pico!!"
- board text added: "I"
- board text added: "LNA"
- board text added: "Pi Pico Rx Copyright (C) Jon Dawson 2023"
- board text added: "Q"

Commit message: Prepare PCB for manufacture
Parts:
- removed C4: 100p, Capacitor_SMD:C_0805_2012Metric
- added R15: 1k, Resistor_SMD:R_0805_2012Metric, F.Cu at (104.1, 150.1)
- added R16: 1k, Resistor_SMD:R_0805_2012Metric, F.Cu at (104.1, 154.9)
- C39: footprint Capacitor_Tantalum_SMD:CP_EIA-7343-31_Kemet-D -> Capacitor_Tantalum_SMD:CP_EIA-3528-21_Kemet-B
- R13, R14: value 1k -> 470
Routing:
- net Net-(U6--): track 22.2 -> 10.3 mm
- net Net-(U5-GPIO26_ADC0): track 35.5 -> 38.5 mm
- net +5V: track 217.3 -> 219.2 mm
- net SPEAKER: track 70.4 -> 71.9 mm
- net Net-(C39-Pad2): track 3.77 -> 5.34 mm
- net Net-(U5-GPIO27_ADC1): track 47.7 -> 48.3 mm
- net GND: track 149.4 -> 148.9 mm, vias 240 -> 238

Commit message: Add gerbers
Parts:
- J5: footprint Connector_Coaxial:SMA_Amphenol_132289_EdgeMount -> Connector_Coaxial:SMA_Samtec_SMA-J-P-X-ST-EM1_EdgeMount
- moved J5 0.79 mm to (115.8, 102.8), turned to 180 degrees
Routing:
- net GND: track 148.9 -> 123.8 mm, vias 238 -> 243
- net Net-(J5-In): track 6.11 -> 6.84 mm
