File: PCB/back_panel/back_panel.kicad_pcb (KiCad board)
At the start: 2 copper layers, 54.6 x 89.5 mm, 4 parts

Commit message: Get CW working
Parts:
- added REF**: OSHW-Logo2_9.8x8mm_SilkScreen, Symbol:OSHW-Logo2_9.8x8mm_SilkScreen, F.Cu at (151.8, 127.0)
Other:
- board text added: "Pi Pico Rx Copyright (C) Jon Dawson 2023"
