File: PCB/Polar_experimental/concept.kicad_sch (KiCad schematic)
At the start: 61 parts, among them J1 Antenna, J2 Speaker, J3 Headphone, J4 SSD1306 I2C Display, J5 Conn_01x08_Pin, J6 Conn_01x07_Pin, J7 Conn_01x03, J8 Conn_01x03, SW1 RotaryEncoder_Switch, SW2 SW_Push, SW3 SW_Push, SW4 SW_Push, U1 MCP6022, U2 Pico, U3 74CBTLV3253, U4 74LVC04

Commit message: latest transceiver experiments
Parts:
- removed C22, C23, C24: 470n, Capacitor_SMD:C_0805_2012Metric, symbol Device:C
- removed R15, R16, R17: 100, Resistor_SMD:R_0805_2012Metric, symbol Device:R
- removed unit 2 of U4
- removed unit 1 of U4
- removed unit 4 of U4
- removed unit 3 of U4
- added U5: 74CBTLV3253, Package_SO:SOIC-16_3.9x9.9mm_P1.27mm, symbol RADIO-rescue:FST5253-xcvr_components
Connections:
- net TX_I is gone; now on net TX_MAGNITUDE: U2.14 (GPIO10)
- net TX_Q is gone; now on net TX_RF: U2.16 (GPIO12)
- net +3V3: now also U5.16 (VCC)
- net DIT: now also SW4.2
- net GND: now also U3.1 (1~{OE}), U5.15 (2~{OE}), U5.2 (S1), U5.5 (1B2), U5.8 (GND)
- net TX_MAGNITUDE: now reaches R14.2
- net at C7.2, R3.2, U3.9 (2A): now also U5.7 (1A); no longer U3.7 (1A)
- net TX_RF: now reaches J6.3 (Pin_3)
- net TX_RF: now also U5.14 (S0)
- net at C21.2, R14.1: now also U5.6 (1B1); no longer U3.5 (1B2)
- removed net PTT: SW4.2, U2.9 (GPIO6), U3.1 (1~{OE})
- new net RX_TX: U2.9 (GPIO6), U5.1 (1~{OE})
- no-connect marks 7 -> 19
Other:
- note added: "Buttons"
- note added: "Quadrature Sampling Detector/Polar Modulator"
- note removed: "Menu Buttons"
- note removed: "Quadrature Sampling Detector/Exciter"
- moved on the sheet: C21, R14, SW1, SW2, SW3, SW4
