File: PCB/QSE_experimental/concept.kicad_sch (KiCad schematic)
At the start: 61 parts, among them J1 Antenna, J2 Speaker, J3 Headphone, J4 SSD1306 I2C Display, J5 Conn_01x08_Pin, J6 Conn_01x07_Pin, J7 Conn_01x03, J8 Conn_01x03, SW1 RotaryEncoder_Switch, SW2 SW_Push, SW3 SW_Push, SW4 SW_Push, U1 MCP6022, U2 Pico, U3 74CBTLV3253, U4 74LVC04

Commit message: latest transceiver experiments
Connections:
- net DIT: now also SW4.2
- net PTT renamed RX_TX
- net RX_TX: no longer SW4.2
Other:
- moved on the sheet: SW1, SW2, SW3, SW4
